File: src/audio-router/transfo_schematic.brd (EAGLE design)
At the start: 54.6 x 72.4 mm, 15 parts

Commit message: v4.3 board design
Parts:
- AMP: value (none) -> TB3POL; device con-phoenix-254:2POL254 -> con-phoenix-381:2POL381
- MIC, SWITCH, TV: value (none) -> TB3POL; device con-phoenix-254:3POL254 -> con-phoenix-381:3POL381
- MICXFMR: value TAMURA-TTC-105-1 -> TTC-105-1
- moved AMP 9.16 mm to (33.0, 19.1)
- moved SWITCH 5.24 mm to (49.5, 6.35)
- moved MIC 5.24 mm to (68.6, 6.35), turned to 180 degrees
- moved TV 4.58 mm to (49.5, 77.5)
- moved R7 2.84 mm to (74.9, 16.5)
- moved R8 2.54 mm to (58.4, 16.5)
- moved MICXFMR 1.27 mm to (66.0, 31.8)
Connections:
- net GND_LIFT renamed TV_GND
- net LEFT renamed TV_LEFT
- net L_LIFT renamed TV_LEFT_LIFT
- net N$1 renamed MIC_HOT
- net PIN2LIFT renamed MIC_HOT_LIFT
- net PIN3LIFT renamed MIC_COLD_LIFT
- net RIGHT renamed TV_RIGHT
- net R_LIFT renamed TV_RIGHT_LIFT
- net TV renamed TV_MONO
- removed net N$2: MIC.3, MICXFMR.P$1, R7.1
- new net MIC_COLD: MIC.1, MICXFMR.P$1, R7.1
- new net MIC_GND: MIC.3, R7.2, R8.1
- net GND: no longer MIC.1, R7.2, R8.1
Routing:
- net MIC_COLD: track 0.00 -> 21.3 mm
- net N$2: track 16.2 -> 0.00 mm
- net TV_GND: track 6.77 -> 0.36 mm
- net MIC_HOT: track 17.3 -> 21.5 mm
- net MIC_HOT_LIFT: track 48.8 -> 52.0 mm
- net AUDIO: track 13.5 -> 16.4 mm
- net TV_RIGHT: track 6.35 -> 8.89 mm
- net TV_LEFT: track 6.77 -> 9.00 mm
- net TV_MONO: track 45.3 -> 45.8 mm
- net MIC_COLD_LIFT: track 15.9 -> 16.4 mm
- added copper zone on layer 16, net MIC_GND
- added copper zone on layer 16, net TV_GND
Other:
- board size 54.6 x 72.4 mm -> 55.9 x 83.8 mm

Commit message: v4.4 board design
Parts:
- removed MICXFMR: TTC-105-1, adam - passive:TAMURA-TTC-105-1
- added T1: TY-311P, TY-311P:XFMR_TY-311P
- moved R4 19.2 mm to (54.6, 47.0), turned to 90 degrees
- moved C1 16.9 mm to (77.5, 47.0), turned to 270 degrees
- moved R3 13.5 mm to (34.3, 47.0), turned to 270 degrees
- moved R9 13.3 mm to (61.0, 47.0), turned to 90 degrees
- moved R10 11.7 mm to (71.1, 47.0), turned to 270 degrees
- moved R1 4.58 mm to (40.6, 47.0), turned to 90 degrees
- moved R2 4.58 mm to (47.0, 47.0), turned to 270 degrees
Connections:
- net GND: now also TR1.6; no longer TR1.4
- net MIC_COLD: now also T1.3; no longer MICXFMR.P$1
- net MIC_COLD_LIFT: now also T1.6; no longer MICXFMR.P$4
- net MIC_HOT: now also T1.1; no longer MICXFMR.P$3
- net MIC_HOT_LIFT: now also T1.4; no longer MICXFMR.P$6
- net TV_LEFT_LIFT: now also R2.1, TR1.5; no longer R1.1, TR1.6
- net TV_MONO: now also R1.1; no longer R1.2
- net TV_RIGHT_LIFT: now also R1.2, TR1.4; no longer R2.1, TR1.5
Routing:
- net TV_LEFT_LIFT: track 16.8 -> 8.45 mm
- net MIC_HOT_LIFT: track 52.0 -> 59.5 mm
- net TV_MONO: track 45.8 -> 51.6 mm
- net MIC_COLD_LIFT: track 16.4 -> 13.8 mm
- net TV_RIGHT_LIFT: track 8.98 -> 11.2 mm
- net MIC_COLD: track 21.3 -> 20.0 mm
- net MIC_HOT: track 21.5 -> 20.2 mm
