File: src/audio-router/transfo_schematic.sch (EAGLE design)
At the start: 15 parts

Commit message: v4.3 board design
Parts:
- AMP: value (none) -> TB3POL; device con-phoenix-254:MPT2 -> con-phoenix-381:MKDS1/2-3,81
- MIC, SWITCH, TV: value (none) -> TB3POL; device con-phoenix-254:MPT3 -> con-phoenix-381:MKDS1/3-3,81
- MICXFMR: value TAMURA-TTC-105-1 -> TTC-105-1
Connections:
- net GND_LIFT renamed TV_GND
- net LEFT renamed TV_LEFT
- net L_LIFT renamed TV_LEFT_LIFT
- net N$1 renamed MIC_HOT
- net PIN2LIFT renamed MIC_HOT_LIFT
- net PIN3LIFT renamed MIC_COLD_LIFT
- net RIGHT renamed TV_RIGHT
- net R_LIFT renamed TV_RIGHT_LIFT
- net TV renamed TV_MONO
- removed net N$2: MIC-3.1, MICXFMR.1, R7.1
- new net MIC_COLD: MIC-1.1, MICXFMR.1, R7.1
- new net MIC_GND: MIC-3.1, R7.2, R8.1
- net GND: no longer MIC-1.1, R7.2, R8.1
Other:
- moved on the sheet: AMP-1, AMP-2, C1, MIC-1, MIC-2, MIC-3, MICXFMR, R1, R10, R2, R3, R4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

Commit message: v4.4 board design
Parts:
- removed MICXFMR: TTC-105-1, adam - passive:TAMURA-TTC-105-1
- added T1: TY-311P, TY-311P:TY-311P
Connections:
- net GND: now also TR1.6; no longer TR1.4
- net MIC_COLD: now also T1.3; no longer MICXFMR.1
- net MIC_COLD_LIFT: now also T1.6; no longer MICXFMR.4
- net MIC_HOT: now also T1.1; no longer MICXFMR.3
- net MIC_HOT_LIFT: now also T1.4; no longer MICXFMR.6
- net TV_LEFT_LIFT: now also R2.1, TR1.5; no longer R1.1, TR1.6
- net TV_MONO: now also R1.1; no longer R1.2
- net TV_RIGHT_LIFT: now also R1.2, TR1.4; no longer R2.1, TR1.5
Other:
- moved on the sheet: R1, R2, R3, TR1, TV-1, TV-2, TV-3
